Commit message: Fixing head servo wrong orientation

File: ros2_ws/src/robotis_mini_description/urdf/body.urdf.xacro (robot description, xacro)
@@ -13,8 +13,4 @@
     <xacro:robotis_mini_lb040 name="body_chest" parent="body_skeleton_link"
         xyz="0 0.016 -0.004" rpy="0 0 0" />
-    <xacro:robotis_mini_servo_rotating_fake name="neck" parent="body_torso_link"
-        xyz="0 0.036 0.006" rpy="${M_PI/2} 0 0" initial_rotation="0" />
-    <xacro:robotis_mini_dmff01 name="body_head" parent="neck_link"
-        xyz="0 0 0.003" rpy="${-M_PI/2} 0 0" />
     <xacro:robotis_mini_spu5 name="l_shoulder_anchor" parent="body_skeleton_link"
         xyz="0.024 0.042 0.009" rpy="${M_PI/2} 0 ${M_PI/2}" />

File: ros2_ws/src/robotis_mini_description/urdf/robotis_mini.urdf.xacro (robot description, xacro)
@@ -13,4 +13,5 @@
   <xacro:include filename="$(find robotis_mini_description)/urdf/hand.urdf.xacro" />
   <xacro:include filename="$(find robotis_mini_description)/urdf/leg.urdf.xacro" />
+  <xacro:include filename="$(find robotis_mini_description)/urdf/head.urdf.xacro" />
   <xacro:robotis_mini_base name="base"/>
   <xacro:robotis_mini_body parent="base_link" />
@@ -19,4 +20,5 @@
   <xacro:robotis_mini_leg side="l" reflect="1" parent="l_hip_anchor_link" />
   <xacro:robotis_mini_leg side="r" reflect="-1" parent="r_hip_anchor_link" />
+  <xacro:robotis_mini_head parent="body_torso_link" />
   <gazebo>
     <plugin name="gazebo_ros_control" filename="libgazebo_ros_control.so">

File: ros2_ws/src/robotis_mini_description/urdf/servo.urdf.xacro (robot description, xacro)
@@ -39,4 +39,5 @@
     <link name="${name}_link">
       <inertial>
+        <origin xyz="0.0 -6.745858e-3 0.697233e-3" rpy="0 0 0" />
         <mass value="0.0001" />
         <inertia ixx="1.0e-12" ixy="0.0" ixz="0.0" iyy="1.0e-12" iyz="0.0" izz="1.0e-12"/>
@@ -53,4 +54,5 @@
     <link name="${name}_axis_link">
       <inertial>
+        <origin xyz="0.0 -6.745858e-3 0.697233e-3" rpy="0 0 0" />
         <mass value="0.0001" />
         <inertia ixx="1.0e-12" ixy="0.0" ixz="0.0" iyy="1.0e-12" iyz="0.0" izz="1.0e-12"/>
@@ -78,4 +80,5 @@
     <link name="${name}_axis_link">
       <inertial>
+        <origin xyz="0.0 -6.745858e-3 0.697233e-3" rpy="0 0 0" />
         <mass value="0.0001" />
         <inertia ixx="1.0e-12" ixy="0.0" ixz="0.0" iyy="1.0e-12" iyz="0.0" izz="1.0e-12"/>
