Commit message: Fixing warnings in webots, caused by a centerOfMass of 0 0 0

File: ros2_ws/src/robotis_mini_description/urdf/common.urdf.xacro (robot description, xacro)
@@ -350,5 +350,5 @@
       </visual>
       <inertial>
-        <origin xyz="0.0 0.0 0.0" rpy="0 0 0" />
+        <origin xyz="-0.000001 0.000001 -0.000001" rpy="0 0 0" />
         <mass value="${MASS_SPD3B3}" />
         <inertia
@@ -380,5 +380,5 @@
       </visual>
       <inertial>
-        <origin xyz="0.0 0.0 0.0" rpy="0 0 0" />
+        <origin xyz="-0.000001 0.000001 -0.000001" rpy="0 0 0" />
         <mass value="${MASS_SPD3B5}" />
         <inertia
@@ -403,5 +403,5 @@
     <link name="${name}_link">
       <visual>
-        <origin xyz="0 0 0" rpy="0 0 0" />
+        <origin xyz="0.0 0.0 0.0" rpy="0 0 0" />
         <geometry>
           <mesh filename="package://robotis_mini_description/meshes/SPD-3B7(W).stl" scale="${STL_SCALE}" />
@@ -410,5 +410,5 @@
       </visual>
       <inertial>
-        <origin xyz="0.0 0.0 0.0" rpy="0 0 0" />
+        <origin xyz="-0.000001 0.000001 -0.000001" rpy="0 0 0" />
         <mass value="${MASS_SPD3B7}" />
         <inertia
@@ -433,5 +433,5 @@
     <link name="${name}_link">
       <visual>
-        <origin xyz="0 0 0" rpy="0 0 0" />
+        <origin xyz="0.0 0.0 0.0" rpy="0 0 0" />
         <geometry>
           <mesh filename="package://robotis_mini_description/meshes/SPD-4B5(W).stl" scale="${STL_SCALE}" />
@@ -440,5 +440,5 @@
       </visual>
       <inertial>
-        <origin xyz="0.0 0.0 0.0" rpy="0 0 0" />
+        <origin xyz="-0.000001 0.000001 -0.000001" rpy="0 0 0" />
         <mass value="${MASS_SPD4B5}" />
         <inertia
@@ -560,5 +560,5 @@
       </visual>
       <inertial>
-        <origin xyz="0.0 0.0 0.0" rpy="0 0 0" />
+        <origin xyz="-0.000001 0.000001 -0.000001" rpy="0 0 0" />
         <mass value="${MASS_LB040}" />
         <inertia

File: ros2_ws/src/robotis_mini_description/urdf/robotis_mini.urdf.xacro (robot description, xacro)
@@ -14,5 +14,5 @@
   <xacro:include filename="$(find robotis_mini_description)/urdf/leg.urdf.xacro" />
   <xacro:include filename="$(find robotis_mini_description)/urdf/head.urdf.xacro" />
-  <xacro:robotis_mini_base name="base"/>
+  <xacro:robotis_mini_base name="base" />
   <xacro:robotis_mini_body parent="base_link" />
   <xacro:robotis_mini_arm side="l" reflect="1" parent="l_shoulder_anchor_link" />
